File: test of knowledge.kicad_pcb (KiCad board)
At the start: 2 copper layers, 55 x 19 mm, 5 parts, among them J1 Screw_Terminal_01x01, J2 Screw_Terminal_01x01, U1 LM7805_TO220

Commit message: Add files via upload
Parts:
- removed J2: Screw_Terminal_01x01, TerminalBlock_Degson:TerminalBlock_Degson_DG250-3.5-01P_1x01_P3.50mm_45Degree
- added C2: 0.1 uF, Capacitor_SMD:C_0805_2012Metric_Pad1.18x1.45mm_HandSolder, F.Cu at (143.0, 76.0)
- added C4: 47uF, Capacitor_SMD:C_Elec_5x5.4, F.Cu at (158.0, 81.0)
- added J3: Screw_Terminal_01x02, TerminalBlock:TerminalBlock_Xinya_XY308-2.54-2P_1x02_P2.54mm_Horizontal, F.Cu at (133.0, 70.0)
- C1: footprint Capacitor_SMD:C_Elec_3x5.4 -> Capacitor_SMD:C_Elec_5x5.4
- J1: value Screw_Terminal_01x01 -> Screw_Terminal_01x02; footprint TerminalBlock_Degson:TerminalBlock_Degson_DG250-3.5-01P_1x01_P3.50mm_45Degree -> TerminalBlock:TerminalBlock_Xinya_XY308-2.54-2P_1x02_P2.54mm_Horizontal
- moved J1 39.6 mm to (162.0, 70.5), turned to 90 degrees
- moved U1 29.1 mm to (144.5, 68.0)
- moved C3 22.8 mm to (151.0, 76.0), turned to 180 degrees
- moved C1 16.1 mm to (138.0, 81.0), turned to 180 degrees
Connections:
- C1 pad 1: Net-(J1-Pin_1) -> Net-(C1-Pad1)
- C1 pad 2: Net-(U1-VI) -> GND
- C3 pad 1: Net-(U1-VO) -> Net-(C3-Pad1)
- C3 pad 2: Net-(J2-Pin_1) -> Net-(U1-VO)
- J1 pad 1: Net-(J1-Pin_1) -> GND
Routing:
- net GND: track 0.00 -> 59.4 mm
- net Net-(J2-Pin_1): track 7.79 -> 0.00 mm
- net Net-(C3-Pad1): track 0.00 -> 6.60 mm
- net Net-(C1-Pad1): track 0.00 -> 5.79 mm
- net Net-(J1-Pin_1): track 5.74 -> 0.00 mm
- net Net-(U1-VI): track 5.92 -> 8.18 mm
- net Net-(U1-VO): track 6.93 -> 8.19 mm
Other:
- board size 55 x 19 mm -> 48 x 26 mm
